File: Files/Hardware/RC2014 - Floppy WD37C65/kicad/RC2014 Floppy WD37C65.kicad_pcb (KiCad board)
At the start: 2 copper layers, 102.5 x 36.8 mm, 18 parts, among them CON1 RC2014, CON2 FLOPPY34, IC1 74HCT138N, IC2 74HCT138N, IC3 74HCT125N, IC4 WD37C65C

Commit message: Some changes
Parts:
- CON1: value RC2014 -> RC2014 Backplane
